Commit message: da installare mimic

File: xacro/arm/ur5_robot.urdf.xacro (robot description, xacro)
@@ -28,5 +28,5 @@
 	</visual>
 	<collision>
-    	<origin xyz="0.0 0.0 0.0" rpy="0.0 0.0 0.0" />
+    	<origin xyz="0.0 0.0 0.0" rpy="0.0 ${-pi/2} 0.0" />
 		<geometry>
 			  <mesh filename="package://progetto_robotica/meshes/gripper/robotiq_85_coupler.stl" />
@@ -46,5 +46,5 @@
     <parent link="world" />
     <child link = "base_link" />
-    <origin xyz="0.0 0.0 1.0" rpy="${pi} 0.0 0.0" />
+    <origin xyz="0.0 0.0 0.0" rpy="0.0 0.0 0.0" />
   </joint>
 </robot>
